File: SOURCES/KICAD/xmos.sch (KiCad schematic (older format))
At the start: 76 parts, among them IC401 IC_NC7WZ07, IC402 NC7SZ175, IC403 IC_XE216-512-TQ128, IC404 IC_CS2100CP, IC405 NC7SZ157, IC406 NC7SZ157, IC407 IC_NCP4681DSQ25T1G, IC408 IC_IS25LP080D, IC409 IC_NCP1117LPST33, IC410 IC_TLV62565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

Commit message: Optimized DAC Output filter
Connections:
- net VDD: now also IC403.78 (VDDIOR)
Changed lines of the file:
@@
 	7250 2450 7250 3350
 Wire Wire Line
-	7250 3350 7250 4950
+	7250 3350 7250 3850
 Wire Wire Line
 	5950 1550 7250 1550
@@
 	5100 8350 5100 8450
 Connection ~ 5100 8450
+Wire Wire Line
+	7100 3850 7250 3850
+Connection ~ 7250 3850
+Wire Wire Line
+	7250 3850 7250 4950
 $EndSCHEMATC
