File: SOURCES/KICAD/ad.sch (KiCad schematic (older format))
At the start: 154 parts, among them IC201 IC_OPA1652AIDR, IC202 IC_OPA1652AIDR, IC203 IC_OPA1652AIDR, IC204 IC_OPA1652AIDR, IC205 IC_AK5558VN, IC206 IC_OPA1652AIDR, IC207 IC_OPA1652AIDR, IC208 IC_OPA1652AIDR, IC209 IC_OPA1652AIDR, X201 CONN_02X13

Commit message: Updated BOM
Parts:
- C201, C202, C209, C210, C215, C216, C225, C226, C235, C236, C245, C246, C253, C254, C267, C268: Manufacturer (none) -> Panasonic Electronic Components; pn (none) -> ECH-U1H102JX5
- C203, C204, C211, C212, C217, C218, C219, C227, C228, C229, C233, C237, C238, C241, C247, C248, C255, C256, C269, C270: Manufacturer (none) -> Nichicon; digikey 399-6102-ND -> UVY1E101MDD-ND; pn (none) -> UVY1E101MDD
- C205, C206, C213, C214, C221, C222, C231, C232, C239, C240, C251, C252, C257, C258, C271, C272: Manufacturer (none) -> KEMET; pn (none) -> C0805C101J5GACTU
- C207, C208, C223, C224, C243, C244, C265, C266: Manufacturer (none) -> Panasonic Electronic Components; pn (none) -> ECH-U1C562JX5
- C220, C230, C234, C242, C249, C261, C262, C264, C273, C274, C275, C276, C277, C278, C279, C280: Manufacturer (none) -> KEMET; pn (none) -> C0805C104K5RACTU
- C250: Manufacturer (none) -> Murata Electronics North America; pn (none) -> GRM21BR61E475MA12L
- C259, C260: Manufacturer (none) -> Murata Electronics North America; pn (none) -> GRM21BR61E106MA73L
- C263: Manufacturer (none) -> Yageo; pn (none) -> CC0805KRX7R9BB103
- IC201, IC202, IC203, IC204, IC206, IC207, IC208, IC209: Manufacturer (none) -> Texas Instruments; pn (none) -> OPA1652AIDR
- IC205: Manufacturer (none) -> AKM Semiconductor Inc.; pn (none) -> AK5558VN
- R201, R202, R207, R208, R219, R220, R229, R230, R240, R241, R247, R248, R253, R254, R259, R260: Manufacturer (none) -> Susumu; pn (none) -> RR1220P-621-D
- R203, R204, R209, R210, R221, R222, R231, R232, R242, R243, R249, R250, R255, R256, R261, R262: Manufacturer (none) -> Susumu; pn (none) -> RR1220P-9760-D-M
- R205, R206, R211, R212, R223, R224, R233, R234, R244, R245, R251, R252, R257, R258, R263, R264: Manufacturer (none) -> Stackpole Electronics Inc.; pn (none) -> RNCP0805FTD10R0
- R213, R214, R215, R216, R217, R235, R236, R237: Manufacturer (none) -> Yageo; pn (none) -> RC0805JR-070RL
- R218, R228, R238, R246: Manufacturer (none) -> Yageo; pn (none) -> RC0805FR-0720RL
- R225, R226, R227: Manufacturer (none) -> Yageo; pn (none) -> RC0805FR-0747KL
- R239: Manufacturer (none) -> Yageo; pn (none) -> RC0805FR-0733RL
- X201: Manufacturer (none) -> Sullins Connector Solutions; pn (none) -> PRPC013DAAN-RC

Commit message: Updated sendParameter
Parts:
- removed C207, C208, C223, C224, C243, C244, C265, C266: CAP_5n60_5%_16V_PPS_0805, rklib:C0805-X7R, symbol rk:CAP_5n60_5%_16V_PPS_0805
- removed C236, C246: CAP_1n00_5%_50V_PPS_0805, rklib:C0805-X7R, symbol rk:CAP_1n00_5%_50V_PPS_0805
- removed C239, C240, C251, C252: CAP_100p_50V_C0G_NP0_0805, rklib:C0805-X7R, symbol rk:CAP_100p_50V_C0G_NP0_0805
- removed R201, R202, R207, R208, R219, R220, R229, R230, R240, R241, R247, R248, R253, R254, R259, R260: RES_620R_0.5%_0.1W_Thin_0805, rklib:C0805-RES, symbol rk:RES_620R_0.5%_0.1W_Thin_0805
- removed R203, R204, R209, R210, R221, R222, R231, R232, R242, R243, R249, R250, R255, R256, R261, R262: RES_976R_0.5%_0.1W_Thin_0805, rklib:C0805-RES, symbol rk:RES_976R_0.5%_0.1W_Thin_0805
- removed R212, R233, R234, R244, R245, R252, R263, R264: RES_10R0_1%_0.25W_Thin_0805, rklib:C0805-RES, symbol rk:RES_10R0_1%_0.25W_Thin_0805
- removed R213, R214, R215, R216, R217, R235, R236, R237: RES_0R00_1%_0.125W_Thick_0805, rklib:C0805-RES, symbol rk:RES_0R00_1%_0.125W_Thick_0805
- removed R225, R226, R227: RES_47K0_1%_0.125W_Thick_0805, rklib:C0805-RES, symbol rk:RES_47K0_1%_0.125W_Thick_0805
- removed X201: CONN_02X13, rklib:HDR_02x13, symbol freeDSP-aurora-rescue:CONN_02X13
- added C207, C208, C223, C224, C239, C251, C265, C266: CAP_220p_2%_50V_PPS_0805, rklib:C0805-X7R, symbol rk:CAP_1n00_5%_50V_PPS_0805
- added C236, C243, C244, C246, C281, C282, C283, C284, C285, C286, C287, C288: CAP_100p_50V_C0G_NP0_0805, rklib:C0805-X7R, symbol rk:CAP_100p_50V_C0G_NP0_0805
- added C240, C252: CAP_1n00_5%_50V_PPS_0805, rklib:C0805-X7R, symbol rk:CAP_1n00_5%_50V_PPS_0805
- added R201, R202, R209, R210, R219, R220, R231, R232, R240, R244, R249, R253, R254, R261, R262, R273: RES_6K80_0.5%_0.125W_Thin_0805, rklib:C0805-RES, symbol rk:RES_10K0_1%_0.25W_Thin_0805
- added R203, R204, R207, R208, R221, R222, R229, R230, R241, R243, R250, R252, R255, R256, R259, R260: RES_10K0_1%_0.25W_Thin_0805, rklib:C0805-RES, symbol rk:RES_10K0_1%_0.25W_Thin_0805
- added R212, R233, R234, R245, R247, R263, R264, R265, R266, R267, R269, R271, R274, R275, R277, R279: RES_2K20_0.5%_0.125W_Thin_0805, rklib:C0805-RES, symbol rk:RES_10K0_1%_0.25W_Thin_0805
- added R242, R248, R268, R270, R272, R276, R278, R280: RES_10R0_1%_0.25W_Thin_0805, rklib:C0805-RES, symbol rk:RES_10R0_1%_0.25W_Thin_0805
- added X201: CON_IDC26, rklib:IDC26, symbol rk:CON_IDC26
- C202, C209, C215, C216, C235, C245, C253, C254: value CAP_1n00_5%_50V_PPS_0805 -> CAP_220p_2%_50V_PPS_0805; Value1 1n00 -> 220p; Value2 5% 50V PPS -> 2% 50V PPS; digikey PCF1328CT-ND -> PCF1288CT-ND; pn ECH-U1H102JX5 -> ECH-U1H221GX5
Connections:
- net +9VA is gone; now on net +5VA: C273.1, C274.1, C275.1, C276.1, C277.1, C278.1, C279.1, C280.1, IC201.8 (V+), IC202.8 (V+), IC203.8 (V+), IC204.8 (V+), IC206.8 (V+), IC207.8 (V+), IC208.8 (V+), IC209.8 (V+)
- net +3V3: now also IC205.44 (CKS1/CAD0_I2C/CSN), IC205.48 (SD/PMOD), IC205.52 (TDM1), IC205.56 (DCKS/HPFE); no longer IC205.53 (PSN/CAD0_SPI)
- net ADC1+: now also C201.2, C213.2, R211.1, R209.1, R265.1; no longer C205.1, R205.1
- net ADC1-: now also C201.1, C205.1, R205.1, R201.1, R266.2; no longer C213.1, R211.1
- net ADC2+: now also C210.2, IC205.63 (AIN2N), C282.2, R210.1, R212.1, R268.1; no longer C206.1, IC205.64 (AIN2P), R206.1
- net ADC2-: now also C206.1, C210.1, IC205.64 (AIN2P), R206.1, R202.1, R267.2; no longer C214.1, IC205.63 (AIN2N)
- net ADC3+: now also C225.2, C283.2, R231.1, R233.1, R270.1; no longer C221.1, R223.1
- net ADC3-: now also C221.1, C225.1, R223.1, R219.1, R269.2; no longer C231.1
- net ADC4+: now also C226.2, IC205.7 (AIN4N), C284.2, R232.1, R234.1, R272.1; no longer C222.1, IC205.8 (AIN4P), R224.1
- net ADC4-: now also C222.1, C226.1, IC205.8 (AIN4P), R224.1, R220.1, R271.2; no longer C232.1, IC205.7 (AIN4N)
- net ADC5+: now also C240.2, C244.2, R244.1, R245.1, R248.1
- net ADC5-: now also C236.1, C240.1, R240.1, R242.1, R247.2; no longer R251.1
- net ADC6+: now also IC205.13 (AIN6N), C252.2, C286.2, R273.1, R274.1, R276.1; no longer IC205.14 (AIN6P)
- net ADC6-: now also IC205.14 (AIN6P), R251.1, C246.1, C252.1, R249.1, R275.2; no longer IC205.13 (AIN6N)
- net ADC7+: now also C267.2, C287.2, R261.1, R263.1, R278.1; no longer C257.1, R257.1
- net ADC7-: now also C257.1, C267.1, R257.1, R253.1, R277.2; no longer C271.1
- net ADC8+: now also C268.2, IC205.21 (AIN8N), C288.2, R262.1, R264.1, R280.1; no longer C258.1, IC205.22 (AIN8P), R258.1
- net ADC8-: now also C258.1, C268.1, IC205.22 (AIN8P), R258.1, R254.1, R279.2; no longer C272.1, IC205.21 (AIN8N)
- net AIN1+: now also C211.2, X201.22 (Pin_22); no longer C203.2
- net AIN1-: now also C203.2, X201.23 (Pin_23); no longer C211.2
- net AIN2+: now also X201.19 (Pin_19)
- net AIN2-: now also X201.20 (Pin_20)
- net AIN3+: now also C227.2, X201.16 (Pin_16); no longer C217.2
- net AIN3-: now also C217.2, X201.17 (Pin_17); no longer C227.2
- net AIN4+: now also X201.13 (Pin_13)
- net AIN4-: now also X201.14 (Pin_14)
- net AIN5+: now also C247.2, X201.10 (Pin_10); no longer C237.2
- net AIN5-: now also C237.2, X201.11 (Pin_11); no longer C247.2
- net AIN6+: now also X201.7 (Pin_7)
- net AIN6-: now also X201.8 (Pin_8)
- net AIN7+: now also C269.2, X201.4 (Pin_4); no longer C255.2
- net AIN7-: now also C255.2, X201.5 (Pin_5); no longer C269.2
- net AIN8+: now also X201.1 (Pin_1)
- net AIN8-: now also X201.2 (Pin_2)
- net GND: now also C213.1, IC205.46 (CKS3/CAD1), IC205.47 (SLOW/DCKB), IC205.49 (DIF0), IC205.50 (DIF1), IC205.51 (TDM0), IC205.53 (PSN/CAD0_SPI), C236.2, C244.1, C246.2, C282.1, C283.1, C284.1, C286.1, C287.1, C288.1, X201.12 (Pin_12), X201.15 (Pin_15), X201.18 (Pin_18), X201.21 (Pin_21), X201.24 (Pin_24), X201.3 (Pin_3), X201.6 (Pin_6), X201.9 (Pin_9); no longer C213.2, C214.2, C231.2, C232.2, C271.2, C272.2
- net VGROUND: no longer IC201.3 (+), IC202.3 (+), IC203.3 (+), IC204.3 (+), IC206.3 (+), IC207.3 (+), IC208.3 (+), IC209.3 (+)
- net at C203.1: now also R207.1
- net at C204.1: now also R208.1
- net at C211.1: now also R203.1
- net at C212.1: now also R204.1
- net at C217.1: now also R229.1
- net at C227.1: now also R221.1
- net at C218.1: now also R230.1
- net at C228.1: now also R222.1
- net at C237.1: now also R243.1
- net at C247.1: now also R241.1
- net at C238.1: now also R252.1
- net at C248.1: now also R250.1
- net at C255.1: now also R259.1
- net at C256.1: now also R260.1
- net at C269.1: now also R255.1
- net at C270.1: now also R256.1
- net at IC201.1, R205.2: now also C207.2; no longer C201.2
- net at IC201.2 (-): now also C207.1, R201.2, R203.2; no longer C201.1
- net at C209.1: now also IC201.3 (+), R207.2, R209.2; no longer IC201.6 (-)
- net at C209.2, IC201.7, R211.2: now also C281.1
- net at C202.1, IC202.2 (-): now also R202.2, R204.2
- net at IC202.6 (-): now also C214.2, R212.2, R267.1; no longer C210.1
- net at IC202.7: now also C214.1, C208.2, R268.2; no longer C210.2
- net at C215.1, IC203.2 (-): now also R219.2, R221.2
- net at IC203.6 (-): now also C231.2, R233.2, R269.1; no longer C225.1
- net at IC203.7: now also C231.1, C223.2, R270.2; no longer C225.2
- net at C216.1, IC204.2 (-): now also R220.2, R222.2
- net at IC204.6 (-): now also C232.2, R234.2, R271.1; no longer C226.1
- net at IC204.7: now also C232.1, C224.2, R272.2; no longer C226.2
- net at C235.2, IC206.1: now also R242.2
- net at C235.1, IC206.2 (-): now also R240.2, R241.2
- net at IC206.6 (-): now also C243.2, R245.2, R247.1; no longer C245.1
- net at C245.2, R251.2: now also IC207.1; no longer IC206.7
- net at IC207.2 (-): now also C245.1, R249.2, R250.2
- net at IC207.6 (-): now also C285.2, R274.2, R275.1
- net at IC207.7: now also C251.2, C285.1, R276.2
- net at C253.1, IC208.2 (-): now also R253.2, R255.2
- net at IC208.6 (-): now also C271.2, R263.2, R277.1; no longer C267.1
- net at IC208.7: now also C271.1, C265.2, R278.2; no longer C267.2
- net at C254.1, IC209.2 (-): now also R254.2, R256.2
- net at IC209.6 (-): now also C272.2, R264.2, R279.1; no longer C268.1
- net at IC209.7: now also C272.1, C266.2, R280.2; no longer C268.2
- net SDA: now reaches IC205.43 (CKS0/SDA/CDTI)
- net SCL: now reaches IC205.45 (CKS2/SCL/CCLK)
- new net: C281.2, IC201.6 (-), R265.2, R266.1
- new net: C265.1, IC208.3 (+), R259.2, R261.2
- new net: C266.1, IC209.3 (+), R260.2, R262.2
- new net: C208.1, IC202.3 (+), R208.2, R210.2
- new net: C223.1, IC203.3 (+), R229.2, R231.2
- new net: C224.1, IC204.3 (+), R230.2, R232.2
- new net: C239.2, C243.1, IC206.7, R248.2
- new net: C239.1, IC206.3 (+), R243.2, R244.2
- new net: C251.1, IC207.3 (+), R252.2, R273.2
Other:
- note added: "I2C addr: 0x22/0x23"
- note removed: "Resistors are only for\nprototype"
- moved on the sheet: C201, C203, C204, C205, C211, C212, C213, C217, C218, C227, C228, C237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
