File: SOURCES/KICAD/da.sch (KiCad schematic (older format))
At the start: 152 parts, among them IC301 IC_OPA1652AIDR, IC302 IC_OPA1652AIDR, IC303 IC_OPA1652AIDR, IC304 IC_OPA1652AIDR, IC305 IC_AK4458VN, IC306 IC_OPA1652AIDR, IC307 IC_OPA1652AIDR, IC308 IC_OPA1652AIDR, IC309 IC_OPA1652AIDR, X301 CONN_02X13

Commit message: Updated sendParameter
Parts:
- removed R359, R360, R361, R362, R363: RES_0R00_1%_0.125W_Thick_0805, rklib:C0805-RES, symbol rk:RES_0R00_1%_0.125W_Thick_0805
- added C370, C371, C372, C373, C374, C375, C376, C377: CAP_100n_50V_X7R_0805, rklib:C0805-X7R, symbol rk:CAP_100n_50V_X7R_0805
- added R374, R375, R376, R377, R378, R379, R380, R381, R382, R383, R384, R385, R386, R387, R388, R389: RES_100K_1%_0.125W_Thick_0805, rklib:C0805-RES, symbol rk:RES_100K_1%_0.125W_Thick_0805
- X301: footprint rklib:HDR_02x13 -> rklib:IDC26; symbol freeDSP-aurora-rescue:CONN_02X13 -> rk:CON_IDC26; digikey ??? -> S2011EC-13-ND
Connections:
- net +9VA is gone; now on net +5VA: C362.1, C363.1, C364.1, C365.1, C366.1, C367.1, C368.1, C369.1, IC301.8 (V+), IC302.8 (V+), IC303.8 (V+), IC304.8 (V+), IC306.8 (V+), IC307.8 (V+), IC308.8 (V+), IC309.8 (V+)
- net +3V3: now also IC305.17 (I2C)
- net AOUT1+: now also C301.2, R374.2; no longer C302.2
- net AOUT1-: now also C309.2, R376.2; no longer C310.2
- net AOUT2+: now also C302.2, R375.2; no longer C301.2
- net AOUT2-: now also C310.2, R377.2; no longer C309.2
- net AOUT3+: now also C315.2, R379.2; no longer C314.2
- net AOUT3-: now also C325.2, R381.2; no longer C324.2
- net AOUT4+: now also C314.2, R378.2; no longer C315.2
- net AOUT4-: now also C324.2, R380.2; no longer C325.2
- net AOUT5+: now also C331.2, R383.2; no longer C330.2
- net AOUT5-: now also C341.2, R385.2; no longer C340.2
- net AOUT6+: now also C330.2, R382.2; no longer C331.2
- net AOUT6-: now also C340.2, R384.2; no longer C341.2
- net AOUT7+: now also C347.2, R387.2; no longer C346.2
- net AOUT7-: now also C357.2, R389.2; no longer C356.2
- net AOUT8+: now also C346.2, R386.2; no longer C347.2
- net AOUT8-: now also C356.2, R388.2; no longer C357.2
- net GND: now also IC305.15 (CAD0_I2C/CSN/_DIF), IC305.16 (PS/CAD0_SPI), C370.2, C371.2, C372.2, C373.2, C374.2, C375.2, C376.2, C377.2, R374.1, R375.1, R376.1, R377.1, R378.1, R379.1, R380.1, R381.1, R382.1, R383.1, R384.1, R385.1, R386.1, R387.1, R388.1, R389.1
- net VGROUND: now also C370.1, C371.1, C372.1, C373.1, C374.1, C375.1, C376.1, C377.1
- net SDA: now reaches IC305.13 (SDA/CDTI/TDM0)
- net SCL: now reaches IC305.14 (SCL/CCLK/TDM1)
Other:
- note added: "I2C addr: 0x20/0x21"
- note removed: "Achtung: Kanäle L/R vertauscht. Im SigmaDSP-Programm berücksichtigen!"
- note removed: "Resistors are only for\nprototype"
- moved on the sheet: C301, C302, C303, C304, C305, C306, C307, C308, C309, C310, C311, C312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
