File: SOURCES/KICAD/freeDSP-aurora.sch (KiCad schematic (older format))
At the start: 76 parts, among them IC101 IC_ADAU1452, IC102 IC_25AA1024, IC103 IC_TLE2426ID, IC104 IC_ADM811TARTZ, IC105 IC_LM1117MP-5.0, IC106 IC_NCP1117LPST33, IC107 IC_LM1117MP-5.0, IC108 IC_LM1117MPX-ADJ, Q101 Q_STD2805, X101 MicroMatch14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

Commit message: Updated sendParameter
Parts:
- removed C112, C114, C137: CAP_10u0_25V_X5R_0805, rklib:C0805-X7R, symbol rk:CAP_10u0_25V_X5R_0805
- removed C113: CAP_100n_50V_X7R_0805, rklib:C0805-X7R, symbol rk:CAP_100n_50V_X7R_0805
- removed IC108: IC_LM1117MPX-ADJ, rklib:SOT223, symbol rk:IC_LM1117MPX-ADJ
- removed R116: RES_150R_1%_0.25W_Thin_0805, rklib:C0805-RES, symbol rk:RES_150R_1%_0.25W_Thin_0805
- removed R117: RES_931R_1%_0.125W_Thick_0805, rklib:C0805-RES, symbol rk:RES_931R_1%_0.125W_Thick_0805
- removed X103: HDR_01x03, rklib:HDR_01x03, symbol freeDSP-aurora-rescue:CONN_01X03
- added C112, C113, C114, C137, C138: CAP_100u_20%_25V_ALUM_RADIAL, rklib:RD2_D5_L11, symbol freeDSP-aurora-rescue:CAP_100u_20%_25V_ALUM_RADIAL
- added R116: RES_560R_1%_0.125W_Thick_0805, rklib:C0805-RES, symbol freeDSP-aurora-rescue:R
- added X103: Conn_01x03, rklib:Molex_PicoBlade_530470310, symbol freeDSP-aurora-rescue:Conn_01x03
- added X106: Conn_01x02, rklib:HDR_01x02, symbol Connector_Generic:Conn_01x02
- B101, B102, B103, B104: Manufacturer (none) -> -; pn (none) -> -
- C101: manf_num GRM21BR61E106MA73L -> (none)
- R101, R102, R104, R105: digikey ??? -> TC164J-33CT-ND
- R108: value 100R -> RES_100R_1%_0.125W_Thick_0805; digikey ??? -> 311-100CRCT-ND
- X101: digikey ??? -> A110871CT-ND
- X102: digikey ??? -> S2011EC-08-ND
- Y101: digikey ??? -> SER3690CT-ND
Connections:
- net +9VA is gone; now on net +5VA: C115.1, C116.1
- net +12V: now also R116.1
- net +3V3: now also X103.1 (Pin_1)
- net +5VA: now also C114.1, C137.1, C138.1
- net AUXADC5: now also X103.2 (Pin_2)
- net GND: now also C112.2, C113.2, C114.2, C137.2, C138.2, X103.3 (Pin_3), X106.2 (Pin_2)
- net VGROUND: now also C112.1, C113.1
- new net: R116.2, X106.1 (Pin_1)
Other:
- moved on the sheet: C111, C115, C116, IC103, X101, X102
