File: SOURCES/KICAD/freeDSP-aurora.sch (KiCad schematic (older format))
At the start: 76 parts, among them IC101 IC_ADAU1452, IC102 IC_25AA1024, IC103 IC_TLE2426ID, IC104 IC_ADM811TARTZ, IC105 IC_LM1117MP-5.0, IC106 IC_NCP1117LPST33, IC107 IC_LM1117MP-5.0, Q101 Q_STD2805, X101 MicroMatch14, X102 HDR_02x08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

Commit message: Note regarding supply voltage
Other:
- note added: "NOTE:\n+12V is the absolute maximum voltage. \n7-7.5V is recommend.\nPlease refer to user manual."
- note removed: "Kondensatoren überprüfen"
- moved on the sheet: X105
Changed lines of the file:
@@
 	1    0    0    -1
 $EndComp
-Text Notes 2000 9900 0    60   ~ 0
-Kondensatoren überprüfen
+Text Notes 1750 9850 0    60   ~ 0
+NOTE:\n+12V is the absolute maximum voltage. \n7-7.5V is recommend.\nPlease refer to user manual.
 $Comp
 L freeDSP-aurora-rescue:GND #PWR054
@@
 L freeDSP-aurora-rescue:+12V #PWR076
 U 1 1 5B82E915
-P 800 9150
-F 0 "#PWR076" H 800 9000 50  0001 C CNN
-F 1 "+12V" H 800 9290 39  0000 C CNN
-F 2 "" H 800 9150 50  0000 C CNN
-F 3 "" H 800 9150 50  0000 C CNN
-	1    800  9150
+P 750 9600
+F 0 "#PWR076" H 750 9450 50  0001 C CNN
+F 1 "+12V" H 750 9740 39  0000 C CNN
+F 2 "" H 750 9600 50  0000 C CNN
+F 3 "" H 750 9600 50  0000 C CNN
+	1    750  9600
 	1    0    0    -1
 $EndComp
@@
 L freeDSP-aurora-rescue:+12V #PWR077
 U 1 1 5B82E91B
-P 1400 9150
-F 0 "#PWR077" H 1400 9000 50  0001 C CNN
-F 1 "+12V" H 1400 9290 39  0000 C CNN
-F 2 "" H 1400 9150 50  0000 C CNN
-F 3 "" H 1400 9150 50  0000 C CNN
-	1    1400 9150
+P 1350 9600
+F 0 "#PWR077" H 1350 9450 50  0001 C CNN
+F 1 "+12V" H 1350 9740 39  0000 C CNN
+F 2 "" H 1350 9600 50  0000 C CNN
+F 3 "" H 1350 9600 50  0000 C CNN
+	1    1350 9600
 	1    0    0    -1
 $EndComp
@@
 L freeDSP-aurora-rescue:GND #PWR078
 U 1 1 5B82E921
-P 800 9350
-F 0 "#PWR078" H 800 9100 50  0001 C CNN
-F 1 "GND" H 800 9200 39  0000 C CNN
-F 2 "" H 800 9350 50  0000 C CNN
-F 3 "" H 800 9350 50  0000 C CNN
-	1    800  9350
+P 750 9800
+F 0 "#PWR078" H 750 9550 50  0001 C CNN
+F 1 "GND" H 750 9650 39  0000 C CNN
+F 2 "" H 750 9800 50  0000 C CNN
+F 3 "" H 750 9800 50  0000 C CNN
+	1    750  9800
 	1    0    0    -1
 $EndComp
@@
 L freeDSP-aurora-rescue:GND #PWR079
 U 1 1 5B82E927
-P 1400 9350
-F 0 "#PWR079" H 1400 9100 50  0001 C CNN
-F 1 "GND" H 1400 9200 39  0000 C CNN
-F 2 "" H 1400 9350 50  0000 C CNN
-F 3 "" H 1400 9350 50  0000 C CNN
-	1    1400 9350
-	1    0    0    -1
-$EndComp
-Wire Wire Line
-	850  9200 800  9200
-Wire Wire Line
-	800  9200 800  9150
-Wire Wire Line
-	850  9300 800  9300
-Wire Wire Line
-	800  9300 800  9350
-Wire Wire Line
-	1350 9200 1400 9200
-Wire Wire Line
-	1400 9200 1400 9150
-Wire Wire Line
-	1350 9300 1400 9300
-Wire Wire Line
-	1400 9300 1400 9350
+P 1350 9800
+F 0 "#PWR079" H 1350 9550 50  0001 C CNN
+F 1 "GND" H 1350 9650 39  0000 C CNN
+F 2 "" H 1350 9800 50  0000 C CNN
+F 3 "" H 1350 9800 50  0000 C CNN
+	1    1350 9800
+	1    0    0    -1
+$EndComp
+Wire Wire Line
+	800  9650 750  9650
+Wire Wire Line
+	750  9650 750  9600
+Wire Wire Line
+	800  9750 750  9750
+Wire Wire Line
+	750  9750 750  9800
+Wire Wire Line
+	1300 9650 1350 9650
+Wire Wire Line
+	1350 9650 1350 9600
+Wire Wire Line
+	1300 9750 1350 9750
+Wire Wire Line
+	1350 9750 1350 9800
 $Comp
 L freeDSP-aurora-rescue:CON_MicroFit3_02x02 X105
 U 1 1 5B82E937
-P 1100 9200
-F 0 "X105" H 1100 9300 39  0000 C CNN
-F 1 "CON_MicroFit3_02x02" H 1100 8900 39  0001 C CNN
-F 2 "rklib:Microfit3_43045-0428" H 1100 8800 39  0001 C CNN
-F 3 "" H 1050 9200 50  0001 C CNN
-F 4 "MicroFit3 02x02" H 1100 9000 39  0000 C CNN "Value1"
-F 5 "WM10670-ND" H 1100 8700 39  0001 C CNN "digikey"
-F 6 "-" H 0   0   50  0001 C CNN "Value2"
-F 7 "Molex, LLC" H 0   0   50  0001 C CNN "Manufacturer"
-F 8 "0430450428" H 0   0   50  0001 C CNN "pn"
-	1    1100 9200
-	1    0    0    -1
-$EndComp
+P 1050 9650
+F 0 "X105" H 1050 9750 39  0000 C CNN
+F 1 "CON_MicroFit3_02x02" H 1050 9350 39  0001 C CNN
+F 2 "rklib:Microfit3_43045-0428" H 1050 9250 39  0001 C CNN
+F 3 "" H 1000 9650 50  0001 C CNN
+F 4 "MicroFit3 02x02" H 1050 9450 39  0000 C CNN "Value1"
+F 5 "WM10670-ND" H 1050 9150 39  0001 C CNN "digikey"
+F 6 "-" H -50 450 50  0001 C CNN "Value2"
+F 7 "Molex, LLC" H -50 450 50  0001 C CNN "Manufacturer"
+F 8 "0430450428" H -50 450 50  0001 C CNN "pn"
+	1    1050 9650
+	1    0    0    -1
+$EndComp
