File: SOURCES/KICAD/freeDSP-aurora DIY.kicad_pcb (KiCad board)
At the start: 2 copper layers, 110 x 110 mm, 505 parts, among them IC101 IC_ADAU1452, IC102 IC_25AA1024, IC103 IC_TLE2426ID, IC104 IC_ADM811TARTZ, IC105 IC_LM1117MP-5.0, IC106 IC_NCP1117LPST33, IC107 IC_LM1117MP-5.0, IC201 IC_OPA1652AIDR, IC202 IC_OPA1652AIDR, IC203 IC_OPA1652AIDR, IC204 IC_OPA1652AIDR, IC205 IC_AK5558VN, IC206 IC_OPA1652AIDR, IC207 IC_OPA1652AIDR, IC208 IC_OPA1652AIDR, IC209 IC_OPA1652AIDR, IC301 IC_OPA1652AIDR, IC302 IC_OPA1652AIDR, IC303 IC_OPA1652AIDR, IC304 IC_OPA1652AIDR, IC305 IC_AK4458VN, IC306 IC_OPA1652AIDR, IC307 IC_OPA1652AIDR, IC308 IC_OPA1652AIDR, IC309 IC_OPA1652AIDR, IC401 IC_NC7WZ07, IC402 NC7SZ175, IC403 IC_XE216-512-TQ128, IC404 IC_CS2100CP, IC405 NC7SZ157, IC406 NC7SZ157, IC407 TLV70025, IC408 IC_IS25LP080D, IC409 IC_NCP1117LPST33, IC410 IC_TLV62565, IC501 ESP32-WROOM-32U, IC502 IC_NCP1117LPST33, Q101 Q_STD2805, SW501 SW_Push, X101 MicroMatch14, X102 HDR_02x08, X103 Conn_01x03, X104 CON_MicroMatch-10G, X105 CON_MicroFit3_02x02, X106 Conn_01x02, X201 CON_IDC26, X301 CON_IDC26, X401 HDR_01x05, X402 CON_HDR_02x10, X501 Conn_01x04, X502 Conn_01x05, X503 Conn_01x03, X504 HDR_01x06, Y101 24M576

Commit message: Bugfix: C124/C125 reversed on silkscreen
Changed lines of the file:
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@@
     (tags 0805)
     (attr smd)
-    (fp_text reference C124 (at -3.5 -1.5 90) (layer F.SilkS)
+    (fp_text reference C124 (at 0 -1.5 90) (layer F.SilkS)
       (effects (font (size 1 1) (thickness 0.15)))
     )
@@
     (tags 0805)
     (attr smd)
-    (fp_text reference C125 (at -3.5 1.5 90) (layer F.SilkS)
+    (fp_text reference C125 (at 0 1.5 90) (layer F.SilkS)
       (effects (font (size 1 1) (thickness 0.15)))
     )
