File: ADDONS/AddOnB/KICAD/Board A/AddOnB.kicad_pcb (KiCad board)
At the start: 2 copper layers, 391 x 45 mm, 136 parts, among them IC1 FIN1002, IC101 74HC251, IC2 FIN1002, IC3 FIN1002, IC4 FIN1002, IC5 IC_NCP1117LPST33, IC6 PCA9536D, SW101 SW_DIP_x08, X1 RCA, X101 XLR3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

Commit message: Bugfix: +3V3 connection on multiplexer
Connections:
- IC101 pad 16: (no net) -> +3V3
Routing:
- net +3V3: track 298.0 -> 300.2 mm
Changed lines of the file:
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@@
-(kicad_pcb (version 20171130) (host pcbnew "(5.0.0-3-g5ebb6b6)")
+(kicad_pcb (version 20171130) (host pcbnew "(5.1.0-0)")
   (general
     (thickness 1.6)
     (drawings 9)
-    (tracks 757)
+    (tracks 759)
     (zones 0)
     (modules 136)
@@
     (zone_45_only no)
     (trace_min 0.2)
-    (segment_width 0.2)
-    (edge_width 0.15)
     (via_size 0.6)
     (via_drill 0.3)
@@
     (uvia_min_size 0.2)
     (uvia_min_drill 0.1)
+    (edge_width 0.15)
+    (segment_width 0.2)
     (pcb_text_width 0.3)
     (pcb_text_size 1.5 1.5)
@@
     (pad 15 smd rect (at 2.7 3.175 90) (size 1.5 0.6) (layers B.Cu B.Paste B.Mask)
       (net 66 "Net-(IC101-Pad15)"))
-    (pad 16 smd rect (at 2.7 4.445 90) (size 1.5 0.6) (layers B.Cu B.Paste B.Mask))
+    (pad 16 smd rect (at 2.7 4.445 90) (size 1.5 0.6) (layers B.Cu B.Paste B.Mask)
+      (net 30 +3V3))
     (model ${KISYS3DMOD}/Package_SO.3dshapes/SOIC-16_3.9x9.9mm_P1.27mm.wrl
       (at (xyz 0 0 0))
@@
   (module rklib:MM-14G (layer F.Cu)
     (at 343.7 -50.2)
-    (fp_text reference X5 (at -0.635 0.5) (layer F.SilkS)
+    (fp_text reference X5 (at 11.1 -1.4) (layer F.SilkS)
       (effects (font (size 1 1) (thickness 0.15)))
     )
@@
   (segment (start 313.1 -61.79) (end 304.71 -53.4) (width 0.6) (layer B.Cu) (net 30))
   (segment (start 313.1 -71.1) (end 313.1 -61.79) (width 0.6) (layer B.Cu) (net 30))
+  (segment (start 329.445 -78.455) (end 329.3 -78.6) (width 0.6) (layer B.Cu) (net 30))
+  (segment (start 329.445 -76.5) (end 329.445 -78.455) (width 0.5) (layer B.Cu) (net 30))
   (segment (start 198.2 -77.45) (end 198.25 -77.5) (width 0.2) (layer B.Cu) (net 31))
   (segment (start 198.2 -75.1) (end 198.2 -77.45) (width 0.2) (layer B.Cu) (net 31))
