File: ADDONS/AddOnB/KICAD/Board A/AddOnB.kicad_pcb (KiCad board)
At the start: 2 copper layers, 391 x 45 mm, 136 parts, among them IC1 FIN1002, IC101 74HC251, IC2 FIN1002, IC3 FIN1002, IC4 FIN1002, IC5 IC_NCP1117LPST33, IC6 PCA9536D, SW101 SW_DIP_x08, X1 RCA, X101 XLR3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

Commit message: Reversed X5
Parts:
- R101, R102, R103, R104, R105, R106, R107, R108, R109, R110, R111, R112, R113, R114, R115, R116: value RES_68R0_1%_0.125W_Thick_0805 -> RES_68R0_1%_0.125W_Thin_0805
Connections:
- net +12V renamed VPP
- X5 pad 1: (no net) -> /SPDIF_RX
- X5 pad 13: /SPDIF_RX -> (no net)
- X5 pad 14: GND -> (no net)
- X5 pad 2: (no net) -> GND
Routing:
- net /SPDIF_RX: track 21.1 -> 34.3 mm
Other:
- board text added: "AddOn-B 1.0.0 auverdion"
- board text removed: "AddOn-B 0.9.0 auverdion"

Commit message: Minor bugfixes on hardware
Changed lines of the file:
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@@
   (page A3)
   (layers
-    (0 F.Cu signal)
+    (0 F.Cu signal hide)
     (31 B.Cu signal)
     (32 B.Adhes user)
@@
     (add_net VPP)
   )
+  (module rklib:Montagewinkel (layer F.Cu)
+    (at 393 -90)
+    (fp_text reference B1 (at 0 0.5) (layer F.SilkS)
+      (effects (font (size 1 1) (thickness 0.15)))
+    )
+    (fp_text value Montagewinkel (at 0 -0.5) (layer F.Fab)
+      (effects (font (size 1 1) (thickness 0.15)))
+    )
+    (fp_line (start -3.5 1) (end 3.5 1) (layer F.SilkS) (width 0.254))
+    (fp_line (start 3.5 0) (end -3.5 0) (layer F.SilkS) (width 0.254))
+    (fp_line (start 3.5 10) (end 3.5 0) (layer F.SilkS) (width 0.254))
+    (fp_line (start -3.5 10) (end 3.5 10) (layer F.SilkS) (width 0.254))
+    (fp_line (start -3.5 0) (end -3.5 10) (layer F.SilkS) (width 0.254))
+    (pad 1 thru_hole circle (at 0 6.5) (size 6 6) (drill 3.2) (layers *.Cu *.Mask))
+  )
   (module rklib:IDC2x8_Pitch2.54mm (layer F.Cu)
     (at 310 -51.16)
@@
     )
   )
-  (module rklib:Montagewinkel (layer F.Cu)
-    (at 393 -90)
-    (fp_text reference B1 (at 0 0.5) (layer F.SilkS)
-      (effects (font (size 1 1) (thickness 0.15)))
-    )
-    (fp_text value Montagewinkel (at 0 -0.5) (layer F.Fab)
-      (effects (font (size 1 1) (thickness 0.15)))
-    )
-    (fp_line (start -3.5 0) (end -3.5 10) (layer F.SilkS) (width 0.254))
-    (fp_line (start -3.5 10) (end 3.5 10) (layer F.SilkS) (width 0.254))
-    (fp_line (start 3.5 10) (end 3.5 0) (layer F.SilkS) (width 0.254))
-    (fp_line (start 3.5 0) (end -3.5 0) (layer F.SilkS) (width 0.254))
-    (fp_line (start -3.5 1) (end 3.5 1) (layer F.SilkS) (width 0.254))
-    (pad 1 thru_hole circle (at 0 7.5) (size 6 6) (drill 3.2) (layers *.Cu *.Mask))
-  )
   (module rklib:KAS2108E (layer F.Cu)
     (at 264 -90 180)
@@
   (segment (start 319.6 -77.85) (end 320.25 -78.5) (width 0.2) (layer B.Cu) (net 90))
   (segment (start 319.6 -76) (end 319.6 -77.85) (width 0.2) (layer B.Cu) (net 90))
-  (segment (start 306.586 -51.114) (end 306.6 -51.1) (width 0.5) (layer B.Cu) (net 102))
-  (segment (start 304.202 -51.114) (end 306.586 -51.114) (width 0.5) (layer B.Cu) (net 102))
-  (segment (start 309.94 -51.1) (end 310 -51.16) (width 0.5) (layer B.Cu) (net 102))
-  (segment (start 306.6 -51.1) (end 309.94 -51.1) (width 0.5) (layer B.Cu) (net 102))
   (segment (start 325.24 -51.16) (end 324.076399 -52.323601) (width 0.2) (layer B.Cu) (net 91))
   (segment (start 317.3 -70.09) (end 317.3 -69.955698) (width 0.2) (layer B.Cu) (net 91))
@@
   (segment (start 267.69 -89) (end 200.120087 -89) (width 0.2) (layer B.Cu) (net 101))
   (segment (start 272.89 -83.8) (end 267.69 -89) (width 0.2) (layer B.Cu) (net 101))
+  (segment (start 306.586 -51.114) (end 306.6 -51.1) (width 0.5) (layer B.Cu) (net 102))
+  (segment (start 304.202 -51.114) (end 306.586 -51.114) (width 0.5) (layer B.Cu) (net 102))
+  (segment (start 309.94 -51.1) (end 310 -51.16) (width 0.5) (layer B.Cu) (net 102))
+  (segment (start 306.6 -51.1) (end 309.94 -51.1) (width 0.5) (layer B.Cu) (net 102))
   (zone (net 17) (net_name GND) (layer F.Cu) (hatch edge 0.508)
     (connect_pads thru_hole_only (clearance 0.2))

Commit message: Updated Gerbers for AddOnB
Parts:
- added REF**: WEEE-Logo_4.2x6mm_SilkScreen, Symbol:WEEE-Logo_4.2x6mm_SilkScreen, B.Cu at (381.0, -50.0)
- added REF**: CE-Logo_8.5x6mm_SilkScreen, Symbol:CE-Logo_8.5x6mm_SilkScreen, B.Cu at (390.0, -50.0)

Commit message: Update AddOnB
Parts:
- moved R101 0.60 mm to (15.3, -69.4)
- moved R102 0.60 mm to (19.1, -69.4)
- moved R103 0.60 mm to (38.3, -69.4)
- moved R104 0.60 mm to (42.1, -69.4)
- moved R107 0.60 mm to (85.2, -68.7)
- moved R108 0.60 mm to (89.0, -68.7)
- moved R109 0.60 mm to (108.2, -68.7)
- moved R110 0.60 mm to (112.0, -68.7)
- moved R111 0.60 mm to (131.2, -68.7)
- moved R112 0.60 mm to (135.0, -68.7)
- moved R113 0.60 mm to (154.2, -68.7)
- moved R114 0.60 mm to (158.0, -68.7)
- moved R115 0.60 mm to (177.2, -68.7)
- moved R116 0.60 mm to (181.0, -68.7)
- moved R105 0.40 mm to (62.2, -68.9)
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Routing:
- net GND: track 98.8 -> 63.4 mm
- net /AOUT2-: track 37.3 -> 43.7 mm
- net /AOUT8+: track 143.2 -> 145.7 mm
- net Net-(R101-Pad2): track 2.22 -> 4.20 mm
- net /AOUT7-: track 129.3 -> 127.9 mm
- net /AOUT3+: track 48.8 -> 50.0 mm
- net /AOUT7+: track 126.2 -> 125.5 mm
- net /AOUT1-: track 21.4 -> 20.8 mm
Other:
- board text added: "AddOn-B 1.0.1 auverdion"
- board text added: "Connect to Analog Input X201"
- board text added: "Connect to Analog Output X301"
- board text removed: "AddOn-B 1.0.0 auverdion"
