File: ADDONS/AddOnC/KICAD/AddOnC.kicad_pcb (KiCad board)
At the start: 2 copper layers, 380 x 45 mm, 97 parts, among them IC102 AK4118AEQ, T101 DA102, T102 DA102, X101 XLR3, X102 XLR3, X103 XLR3, X104 XLR3, X105 XLR3, X106 XLR3, X107 XLR3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

Commit message: Production files AddOn C
Parts:
- X112: value USB_A -> HDR_01x05; footprint Connector_USB:USB_A_CNCTech_1001-011-01101_Horizontal -> Connector_PinHeader_2.54mm:PinHeader_1x05_P2.54mm_Vertical
- moved X112 6.51 mm to (274.3, -46.9), turned to 90 degrees
- moved X5 1.00 mm to (259.8, -48.8)
Routing:
- net Net-(X111-Pad4): track 29.9 -> 39.3 mm
- net +3V3: track 214.8 -> 218.8 mm
- net /D+: track 29.9 -> 33.5 mm
- net /D-: track 30.1 -> 33.5 mm
- net /OPTICAL_RX: track 31.8 -> 34.2 mm
- net Net-(X111-Pad1): track 36.1 -> 34.2 mm
- net +5V: track 41.1 -> 42.1 mm
Other:
- board text added: "AddOn C 0.9.0 auverdion"
- board text removed: "AddOn-C 0.9.0 auverdion"
