File: ADDONS/AddOnC/KICAD/AddOnC.sch (KiCad schematic (older format))
At the start: 97 parts, among them IC102 AK4118AEQ, T101 DA102, T102 DA102, X101 XLR3, X102 XLR3, X103 XLR3, X104 XLR3, X105 XLR3, X106 XLR3, X107 XLR3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

Commit message: Production files AddOn C
Parts:
- removed X112: USB_A, Connector_USB:USB_A_CNCTech_1001-011-01101_Horizontal, symbol Connector:USB_A
- added X112: HDR_01x05, Connector_PinHeader_2.54mm:PinHeader_1x05_P2.54mm_Vertical, symbol Connector_Generic:Conn_01x05
Connections:
- wire segments 351 -> 355
Changed lines of the file:
@@
 	1    0    0    -1
 $EndComp
-$Comp
-L Connector:USB_A X112
-U 1 1 5FD213FB
-P 12900 8200
-F 0 "X112" H 12950 8600 39  0000 R CNN
-F 1 "USB_A" H 13000 8550 39  0000 R CNN
-F 2 "Connector_USB:USB_A_CNCTech_1001-011-01101_Horizontal" H 13050 8150 50  0001 C CNN
-F 3 " ~" H 13050 8150 50  0001 C CNN
-	1    12900 8200
-	-1   0    0    -1
-$EndComp
-Wire Wire Line
-	12400 8000 12600 8000
-Wire Wire Line
-	12400 8200 12600 8200
-Wire Wire Line
-	12400 8300 12600 8300
 Wire Wire Line
 	12100 8600 12100 8650
 Wire Wire Line
-	12100 8650 12900 8650
-Wire Wire Line
-	12900 8650 12900 8600
+	12100 8650 12950 8650
 Wire Wire Line
 	12000 8600 12000 8750
 Wire Wire Line
 	12000 8750 13000 8750
-Wire Wire Line
-	13000 8750 13000 8600
 Text Label 12450 8200 0    39   ~ 0
 D+
@@
 USB_SHIELD
 NoConn ~ 10500 10550
+$Comp
+L Connector_Generic:Conn_01x05 X112
+U 1 1 5E1CADC4
+P 13250 8200
+F 0 "X112" H 13330 8234 39  0000 L CNN
+F 1 "HDR_01x05" H 13330 8159 39  0000 L CNN
+F 2 "Connector_PinHeader_2.54mm:PinHeader_1x05_P2.54mm_Vertical" H 13250 8200 50  0001 C CNN
+F 3 "~" H 13250 8200 50  0001 C CNN
+	1    13250 8200
+	1    0    0    -1
+$EndComp
+Wire Wire Line
+	12400 8000 13050 8000
+Wire Wire Line
+	12400 8200 13050 8200
+Wire Wire Line
+	13000 8400 13050 8400
+Wire Wire Line
+	13000 8400 13000 8750
+Wire Wire Line
+	13050 8300 12950 8300
+Wire Wire Line
+	12950 8300 12950 8650
+Wire Wire Line
+	12900 8300 12900 8100
+Wire Wire Line
+	12900 8100 13050 8100
+Wire Wire Line
+	12400 8300 12900 8300
 $EndSCHEMATC
