File: ADDONS/AddOnB/KICAD/Board B/AddOnB.kicad_pcb (KiCad board)
At the start: 2 copper layers, 189 x 36 mm, 57 parts, among them X101 XLR3, X102 XLR3, X103 XLR3, X104 XLR3, X105 XLR3, X106 XLR3, X107 XLR3, X108 XLR3, X109 CON_IDC26

Commit message: Schematic AddOn-A
Parts:
- added R133: RES_7K87_0.5%_0.100W_Thin_0805, rklib:C0805-RES, B.Cu at (34.0, -70.0)
- added R134: RES_5K11_0.5%_0.100W_Thin_0805, rklib:C0805-RES, B.Cu at (36.0, -70.0)
- added R135: RES_7K87_0.5%_0.100W_Thin_0805, rklib:C0805-RES, B.Cu at (32.0, -70.0)
- added R136: RES_7K87_0.5%_0.100W_Thin_0805, rklib:C0805-RES, B.Cu at (49.0, -70.0)
- added R137: RES_5K11_0.5%_0.100W_Thin_0805, rklib:C0805-RES, B.Cu at (48.0, -67.2)
- added R138: RES_7K87_0.5%_0.100W_Thin_0805, rklib:C0805-RES, B.Cu at (47.0, -70.0)
- added R139: RES_7K87_0.5%_0.100W_Thin_0805, rklib:C0805-RES, B.Cu at (68.0, -70.0)
- added R140: RES_5K11_0.5%_0.100W_Thin_0805, rklib:C0805-RES, B.Cu at (67.0, -67.2)
- added R141: RES_7K87_0.5%_0.100W_Thin_0805, rklib:C0805-RES, B.Cu at (66.0, -70.0)
- added R142: RES_7K87_0.5%_0.100W_Thin_0805, rklib:C0805-RES, B.Cu at (82.9, -70.0)
- added R143: RES_5K11_0.5%_0.100W_Thin_0805, rklib:C0805-RES, B.Cu at (78.9, -70.0)
- added R144: RES_7K87_0.5%_0.100W_Thin_0805, rklib:C0805-RES, B.Cu at (80.9, -70.0)
- added R145: RES_7K87_0.5%_0.100W_Thin_0805, rklib:C0805-RES, B.Cu at (106.0, -70.0)
- added R146: RES_5K11_0.5%_0.100W_Thin_0805, rklib:C0805-RES, B.Cu at (102.0, -70.0)
- added R147: RES_7K87_0.5%_0.100W_Thin_0805, rklib:C0805-RES, B.Cu at (104.0, -70.0)
- added R148: RES_7K87_0.5%_0.100W_Thin_0805, rklib:C0805-RES, B.Cu at (129.0, -70.0)
- added R149: RES_5K11_0.5%_0.100W_Thin_0805, rklib:C0805-RES, B.Cu at (125.0, -70.0)
- added R150: RES_7K87_0.5%_0.100W_Thin_0805, rklib:C0805-RES, B.Cu at (127.0, -70.0)
- added R151: RES_7K87_0.5%_0.100W_Thin_0805, rklib:C0805-RES, B.Cu at (152.0, -70.0)
- added R152: RES_5K11_0.5%_0.100W_Thin_0805, rklib:C0805-RES, B.Cu at (148.0, -70.0)
- added R153: RES_7K87_0.5%_0.100W_Thin_0805, rklib:C0805-RES, B.Cu at (150.0, -70.0)
- added R154: RES_7K87_0.5%_0.100W_Thin_0805, rklib:C0805-RES, B.Cu at (175.0, -70.0)
- added R155: RES_5K11_0.5%_0.100W_Thin_0805, rklib:C0805-RES, B.Cu at (171.0, -70.0)
- added R156: RES_7K87_0.5%_0.100W_Thin_0805, rklib:C0805-RES, B.Cu at (173.0, -70.0)
- moved C106 4.00 mm to (62.0, -70.0)
- moved R111 4.00 mm to (64.0, -70.0)
- moved R112 4.00 mm to (60.0, -70.0)
- moved C103 2.00 mm to (53.0, -70.0)
- moved C104 2.00 mm to (43.0, -70.0)
- moved R105 2.00 mm to (51.0, -70.0)
- moved R106 2.00 mm to (55.0, -70.0)
- moved R107 2.00 mm to (41.0, -70.0)
- moved R108 2.00 mm to (45.0, -70.0)
- moved X102 0.10 mm to (43.1, -90.0)
- moved X103 0.10 mm to (66.1, -90.0)
Connections:
- C101 pad 1: /AIN1+ -> Net-(C101-Pad1)
- C102 pad 1: /AIN1- -> Net-(C102-Pad1)
- C103 pad 1: /AIN2+ -> Net-(C103-Pad1)
- C104 pad 1: /AIN2- -> Net-(C104-Pad1)
- C105 pad 1: /AIN3+ -> Net-(C105-Pad1)
- C106 pad 1: /AIN3- -> Net-(C106-Pad1)
- C107 pad 1: /AIN4+ -> Net-(C107-Pad1)
- C108 pad 1: /AIN4- -> Net-(C108-Pad1)
- C109 pad 1: /AIN5+ -> Net-(C109-Pad1)
- C110 pad 1: /AIN5- -> Net-(C110-Pad1)
- C111 pad 1: /AIN6+ -> Net-(C111-Pad1)
- C112 pad 1: /AIN6- -> Net-(C112-Pad1)
- C113 pad 1: /AIN7+ -> Net-(C113-Pad1)
- C114 pad 1: /AIN7- -> Net-(C114-Pad1)
- C115 pad 1: /AIN8+ -> Net-(C115-Pad1)
- C116 pad 1: /AIN8- -> Net-(C116-Pad1)
- R101 pad 2: /AIN1+ -> Net-(C101-Pad1)
- R102 pad 2: /AIN1+ -> Net-(C101-Pad1)
- R103 pad 2: /AIN1- -> Net-(C102-Pad1)
- R104 pad 2: /AIN1- -> Net-(C102-Pad1)
- R105 pad 2: /AIN2+ -> Net-(C103-Pad1)
- R106 pad 2: /AIN2+ -> Net-(C103-Pad1)
- R107 pad 2: /AIN2- -> Net-(C104-Pad1)
- R108 pad 2: /AIN2- -> Net-(C104-Pad1)
- R109 pad 2: /AIN3+ -> Net-(C105-Pad1)
- R110 pad 2: /AIN3+ -> Net-(C105-Pad1)
- R111 pad 2: /AIN3- -> Net-(C106-Pad1)
- R112 pad 2: /AIN3- -> Net-(C106-Pad1)
- R113 pad 2: /AIN4+ -> Net-(C107-Pad1)
- R114 pad 2: /AIN4+ -> Net-(C107-Pad1)
- R115 pad 2: /AIN4- -> Net-(C108-Pad1)
- R116 pad 2: /AIN4- -> Net-(C108-Pad1)
- R117 pad 2: /AIN5+ -> Net-(C109-Pad1)
- R118 pad 2: /AIN5+ -> Net-(C109-Pad1)
- R119 pad 2: /AIN5- -> Net-(C110-Pad1)
- R120 pad 2: /AIN5- -> Net-(C110-Pad1)
- R121 pad 2: /AIN6+ -> Net-(C111-Pad1)
- R122 pad 2: /AIN6+ -> Net-(C111-Pad1)
- R123 pad 2: /AIN6- -> Net-(C112-Pad1)
- R124 pad 2: /AIN6- -> Net-(C112-Pad1)
- R125 pad 2: /AIN7+ -> Net-(C113-Pad1)
- R126 pad 2: /AIN7+ -> Net-(C113-Pad1)
- R127 pad 2: /AIN7- -> Net-(C114-Pad1)
- R128 pad 2: /AIN7- -> Net-(C114-Pad1)
- R129 pad 2: /AIN8+ -> Net-(C115-Pad1)
- R130 pad 2: /AIN8+ -> Net-(C115-Pad1)
- R131 pad 2: /AIN8- -> Net-(C116-Pad1)
- R132 pad 2: /AIN8- -> Net-(C116-Pad1)
Routing:
- net Net-(C107-Pad1): track 0.00 -> 14.1 mm
- net Net-(C109-Pad1): track 0.00 -> 12.7 mm
- net Net-(C102-Pad1): track 0.00 -> 12.7 mm
- net Net-(C115-Pad1): track 0.00 -> 12.7 mm
- net Net-(C113-Pad1): track 0.00 -> 12.7 mm
- net Net-(C111-Pad1): track 0.00 -> 12.7 mm
- net /AIN1-: track 41.6 -> 29.4 mm
- net /AIN4+: track 30.5 -> 19.2 mm
- net /AIN5+: track 52.5 -> 41.2 mm
- net /AIN7+: track 90.8 -> 79.5 mm
- net /AIN8+: track 107.5 -> 96.2 mm
- net /AIN6+: track 68.8 -> 57.5 mm
- net Net-(C108-Pad1): track 0.00 -> 11.1 mm
- net /AIN4-: track 30.6 -> 21.0 mm
- net Net-(C110-Pad1): track 0.00 -> 8.90 mm
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
Commit message: Updated XLR input board of AddOnB
Parts:
- added REF**: WEEE-Logo_5.6x8mm_SilkScreen, Symbol:WEEE-Logo_5.6x8mm_SilkScreen, B.Cu at (188.0, -60.0)
- added REF**: CE-Logo_8.5x6mm_SilkScreen, Symbol:CE-Logo_8.5x6mm_SilkScreen, B.Cu at (179.0, -60.0)
Other:
- board size 189 x 36 mm -> 186 x 36 mm
- board text added: "XLR Input Board auverdion 1.0.0"
- board text removed: "AddOn-B 0.9.0 auverdion"
