File: ADDONS/AddOnB/KICAD/Board B/AddOnB.sch (KiCad schematic (older format))
At the start: 57 parts, among them X101 XLR3, X102 XLR3, X103 XLR3, X104 XLR3, X105 XLR3, X106 XLR3, X107 XLR3, X108 XLR3, X109 CON_IDC26

Commit message: Schematic AddOn-A
Parts:
- added R133, R135, R136, R138, R139, R141, R142, R144, R145, R147, R148, R150, R151, R153, R154, R156: RES_7K87_0.5%_0.100W_Thin_0805, rklib:C0805-RES, symbol rk:RES_0R00_1%_0.125W_Thick_0805
- added R134, R137, R140, R143, R146, R149, R152, R155: RES_5K11_0.5%_0.100W_Thin_0805, rklib:C0805-RES, symbol rk:RES_0R00_1%_0.125W_Thick_0805
- C101, C102, C103, C104, C105, C106, C107, C108, C109, C110, C111, C112, C113, C114, C115, C116: Manufacturer (none) -> Kemet; pn (none) -> C0805C101J5GACTU
- R101, R103, R105, R107, R109, R111, R113, R115, R117, R119, R121, R123, R125, R127, R129, R131: pn (none) -> RNCP0805FTD100R
- R102, R104, R106, R108, R110, R112, R114, R116, R118, R120, R122, R124, R126, R128, R130, R132: pn (none) -> RC0805FR-07100KL
Connections:
- net AIN1+: now also R133.2, R134.2; no longer C101.1, R101.2, R102.2
- net AIN1-: now also R134.1, R135.2; no longer C102.1, R103.2, R104.2
- net AIN2+: now also R136.2, R137.2; no longer C103.1, R105.2, R106.2
- net AIN2-: now also R137.1, R138.2; no longer C104.1, R107.2, R108.2
- net AIN3+: now also R139.2, R140.2; no longer C105.1, R109.2, R110.2
- net AIN3-: now also R140.1, R141.2; no longer C106.1, R111.2, R112.2
- net AIN4+: now also R142.2, R143.2; no longer C107.1, R113.2, R114.2
- net AIN4-: now also R143.1, R144.2; no longer C108.1, R115.2, R116.2
- net AIN5+: now also R145.2, R146.2; no longer C109.1, R117.2, R118.2
- net AIN5-: now also R146.1, R147.2; no longer C110.1, R119.2, R120.2
- net AIN6+: now also R148.2, R149.2; no longer C111.1, R121.2, R122.2
- net AIN6-: now also R149.1, R150.2; no longer C112.1, R123.2, R124.2
- net AIN7+: now also R151.2, R152.2; no longer C113.1, R125.2, R126.2
- net AIN7-: now also R152.1, R153.2; no longer C114.1, R127.2, R128.2
- net AIN8+: now also R154.2, R155.2; no longer C115.1, R129.2, R130.2
- net AIN8-: now also R155.1, R156.2; no longer C116.1, R131.2, R132.2
- new net: C101.1, R101.2, R102.2, R133.1
- new net: C102.1, R103.2, R104.2, R135.1
- new net: C103.1, R105.2, R106.2, R136.1
- new net: C104.1, R107.2, R108.2, R138.1
- new net: C105.1, R109.2, R110.2, R139.1
- new net: C106.1, R111.2, R112.2, R141.1
- new net: C107.1, R113.2, R114.2, R142.1
- new net: C108.1, R115.2, R116.2, R144.1
- new net: C109.1, R117.2, R118.2, R145.1
- new net: C110.1, R119.2, R120.2, R147.1
- new net: C111.1, R121.2, R122.2, R148.1
- new net: C112.1, R123.2, R124.2, R150.1
- new net: C113.1, R125.2, R126.2, R151.1
- new net: C114.1, R127.2, R128.2, R153.1
- new net: C115.1, R129.2, R130.2, R154.1
- new net: C116.1, R131.2, R132.2, R156.1

Commit message: Updated BOM AddOnB
Parts:
- R101, R103, R105, R107, R109, R111, R113, R115, R117, R119, R121, R123, R125, R127, R129, R131: Manufacturer (none) -> Susumu
- R102, R104, R106, R108, R110, R112, R114, R116, R118, R120, R122, R124, R126, R128, R130, R132: Manufacturer (none) -> Yageo
- R133, R135, R136, R138, R139, R141, R142, R144, R145, R147, R148, R150, R151, R153, R154, R156: value RES_7K87_0.5%_0.100W_Thin_0805 -> RES_0R00_1%_0.125W_Thick_0805; Manufacturer Susumu -> Yageo; Value1 7K87 -> 0R00; Value2 0.5% 0.100W Thin -> 0.5% 0.125W Thick; digikey RR12P7.87KDCT-ND -> (none); pn RR1220P-7871-D-M -> RC0805FR-070RL
- R134, R137, R140, R143, R146, R149, R152, R155: value RES_5K11_0.5%_0.100W_Thin_0805 -> RES_DNP; Manufacturer Susumu -> (none); Value1 5K11 -> (none); Value2 0.5% 0.100W Thin -> (none); digikey RR12P5.11KDCT-ND -> (none); pn RR1220P-5111-D-M -> (none)
- X101, X102, X103, X104, X105, X106, X107, X108: Manufacturer (none) -> Neutrik; pn (none) -> NC3FAH1
- X109: Manufacturer (none) -> Bud Industries; pn (none) -> BC-32677

Commit message: PDF schematic AddOn B
Other:
- note added: "Connect to X201 on Aurora mainboard\nand to X114 on Board A.\nDaisy chain X109 -> X114 -> X201\nor X114 -> X109 -> X201"
Changed lines of the file:
@@
 EESchema Schematic File Version 4
-LIBS:AddOnB-cache
-EELAYER 29 0
+EELAYER 30 0
 EELAYER END
 $Descr A3 16535 11693
 encoding utf-8
 Sheet 1 1
-Title ""
+Title "Addon B Board B"
 Date ""
 Rev ""
-Comp ""
+Comp "auverdion"
 Comment1 ""
 Comment2 ""
@@
 Wire Wire Line
 	4650 10400 4850 10400
+Text Notes 8300 5850 0    79   ~ 0
+Connect to X201 on Aurora mainboard\nand to X114 on Board A.\nDaisy chain X109 -> X114 -> X201\nor X114 -> X109 -> X201
 $EndSCHEMATC

Commit message: Updated XLR input board of AddOnB
Parts:
- R101, R103, R105, R107, R109, R111, R113, R115, R117, R119, R121, R123, R125, R127, R129, R131: symbol rk:RES_100R_1%_0.25W_Thin_0805 -> AddOnB-rescue:RES_100R_1%_0.25W_Thin_0805-rk; pn RNCP0805FTD100R -> RR1220P-101-D
- R133, R135, R136, R138, R139, R141, R142, R144, R145, R147, R148, R150, R151, R153, R154, R156: digikey (none) -> RR12P7.87KDCT-ND; pn RC0805FR-070RL -> RC0805JR-070RL
- R134, R137, R140, R143, R146, R149, R152, R155: Value1 (none) -> DNP; digikey (none) -> RR12P5.11KDCT-ND
Other:
- note removed: "Connect to X201 on Aurora mainboard\nand to X114 on Board A.\nDaisy chain X109 -> X114 -> X201\nor X114 -> X109 -> X201"
